Commit message: tracker and sim stuff

File: Python/Daniel/models/mri/urdf/mri.urdf (robot description, URDF)
Before this commit: robot mri, 1 links, 0 joints
Links:
- link base_link: geometry collision mesh filename=package://mri/meshes/base_link.STL; visual mesh filename=package://mri/meshes/base_link.STL

File: Python/Daniel/models/mri/urdf/mri_vhacd.urdf (robot description, URDF)
Before this commit: robot mri, 1 links, 0 joints
Links:
- link base_link: geometry collision mesh filename=/home/daniel/Desktop/robotPathPlanning/Python/Daniel/models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; visual mesh filename=/home/daniel/Desktop/robotPathPlanning/Python/Daniel/models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
